File: electronics/encoder_can_v2/encoder_can_v2.kicad_sch (KiCad schematic)
At the start: 33 parts, among them J1 5V GND CANH CANL solder pads, J2 SWD pogo P2.54, U1 STM32G431KBU6, U2 TMAG5273A2QDBVR, U3 TMAG5273A2QDBVR, U4 TCAN332GDCNR, U5 TPS7A2033PDBVR, Y1 16MHz CL12pF ESR80

Commit message: Save CAN encoder V2.4 for D70 reducer geometry
Preserve the narrow four-layer 0.8 mm PCB with fixed Hall positions, 0.5 mm via-to-pad clearance and vias outside component bodies. Record the D70 reducer dimensions and variant identifier explicitly.

Include matching manufacturing files, assembly data, release audits and the mechanical generator integration. Validate with 23 generator tests and zero native ERC, DRC, unconnected and schematic parity errors after unpacking the portable project. Keep ZIP and STL deliverables outside Git.
Parts:
- added D2: LED green, Encoder_CAN:LED_Kingbright_APG1005, symbol Device:LED
- added D3: LED yellow, Encoder_CAN:LED_Kingbright_APG1005, symbol Device:LED
- added D4: LED red, Encoder_CAN:LED_Kingbright_APG1005, symbol Device:LED
- added R10, R11, R12: 1k, Encoder_CAN:R_0402_Status, symbol Device:R
Connections:
- net +3V3: now also R10.1
- net GND: now also D2.1 (K), D3.1 (K), D4.1 (K)
- net LED_PHASE: now reaches U1.10 (PA5)
- net LED_PHASE: now also R12.1
- net LED_CMD: now reaches U1.9 (PA4)
- net LED_CMD: now also R11.1
- new net LED_CMD_A: D3.2 (A), R11.2
- new net LED_PHASE_A: D4.2 (A), R12.2
- new net LED_PWR_A: D2.2 (A), R10.2
- no-connect marks 15 -> 13
